File: PTL-IR_remote.sch (KiCad schematic (older format))
At the start: 15 parts, among them J1 8p, J2 8p, Q1 2N7002, U1 TSOP45xx

Commit message: add correction notes on schema
Parts:
- renumbered PR to PR1
Other:
- note added: "Corriger plan de masse"
- note added: "Ev version pass through\n"
- note added: "Passer sensors en 3V3"
- note added: "mesurer tension sur pin data IRM"
Changed lines of the file:
@@
 	5050 2750 5050 2650
 $Comp
-L R_PHOTO PR
+L R_PHOTO PR1
 U 1 1 5B48DA29
 P 3050 4100
-F 0 "PR" H 3100 4150 50  0000 L CNN
+F 0 "PR1" H 3100 4150 50  0000 L CNN
 F 1 "PHOTO" H 3100 4100 50  0000 L TNN
 F 2 "Socket_Strips:Socket_Strip_Straight_1x02_Pitch2.54mm" V 3100 3850 50  0001 L CNN
@@
 	1    0    0    -1
 $EndComp
+Text Notes 8250 950  0    60   ~ 0
+Passer sensors en 3V3
+Text Notes 8250 1100 0    60   ~ 0
+Corriger plan de masse
+Text Notes 8250 1300 0    60   ~ 0
+Ev version pass through\n
+Text Notes 8250 1500 0    60   ~ 0
+mesurer tension sur pin data IRM
 $EndSCHEMATC

Commit message: anotate schema modifs
Parts:
- PR1: value PHOTO -> PHOTO (1MΩ)
- R1: value 1kΩ -> 1kΩ (10kΩ)
Other:
- note added: "Annoter certaines pins (5V, 3V3, GND,...)"
- note added: "C1 en 0603 et R aussi"
- note added: "LED RGB WS2812 WS2813"
- note added: "enlever bme280"
Changed lines of the file:
@@
 P 3050 4100
 F 0 "PR1" H 3100 4150 50  0000 L CNN
-F 1 "PHOTO" H 3100 4100 50  0000 L TNN
+F 1 "PHOTO (1MΩ)" H 3100 4100 50  0000 L TNN
 F 2 "Socket_Strips:Socket_Strip_Straight_1x02_Pitch2.54mm" V 3100 3850 50  0001 L CNN
 F 3 "" H 3050 4050 50  0001 C CNN
@@
 P 3050 4650
 F 0 "R1" V 3130 4650 50  0000 C CNN
-F 1 "1kΩ" V 2950 4650 50  0000 C CNN
+F 1 "1kΩ (10kΩ)" V 2950 4650 50  0000 C CNN
 F 2 "Resistors_SMD:R_1206" V 2980 4650 50  0001 C CNN
 F 3 "" H 3050 4650 50  0001 C CNN
@@
 	1    0    0    -1
 $EndComp
-$Comp
-L +5V #PWR08
-U 1 1 5B48FB68
-P 8300 4600
-F 0 "#PWR08" H 8300 4450 50  0001 C CNN
-F 1 "+5V" H 8300 4740 50  0000 C CNN
-F 2 "" H 8300 4600 50  0001 C CNN
-F 3 "" H 8300 4600 50  0001 C CNN
-	1    8300 4600
-	1    0    0    -1
-$EndComp
 Wire Wire Line
 	6200 4850 6200 5100
@@
 Text Label 4900 4550 0    60   ~ 0
 D5
-$Comp
-L +5V #PWR09
-U 1 1 5B490AA6
-P 6100 2650
-F 0 "#PWR09" H 6100 2500 50  0001 C CNN
-F 1 "+5V" H 6100 2790 50  0000 C CNN
-F 2 "" H 6100 2650 50  0001 C CNN
-F 3 "" H 6100 2650 50  0001 C CNN
-	1    6100 2650
-	1    0    0    -1
-$EndComp
 Wire Wire Line
 	6100 2750 6100 2650
 $Comp
-L +3.3V #PWR010
+L +3.3V #PWR08
 U 1 1 5B490C6C
 P 3050 3700
-F 0 "#PWR010" H 3050 3550 50  0001 C CNN
+F 0 "#PWR08" H 3050 3550 50  0001 C CNN
 F 1 "+3.3V" H 3050 3840 50  0000 C CNN
 F 2 "" H 3050 3700 50  0001 C CNN
@@
 	8300 4650 8550 4650
 $Comp
-L +5V #PWR011
+L +5V #PWR09
 U 1 1 5B490F29
 P 6650 4950
-F 0 "#PWR011" H 6650 4800 50  0001 C CNN
+F 0 "#PWR09" H 6650 4800 50  0001 C CNN
 F 1 "+5V" H 6650 5090 50  0000 C CNN
 F 2 "" H 6650 4950 50  0001 C CNN
@@
 $EndComp
 $Comp
-L +3.3V #PWR012
+L +3.3V #PWR010
 U 1 1 5B490F5E
 P 3800 4750
-F 0 "#PWR012" H 3800 4600 50  0001 C CNN
+F 0 "#PWR010" H 3800 4600 50  0001 C CNN
 F 1 "+3.3V" H 3800 4890 50  0000 C CNN
 F 2 "" H 3800 4750 50  0001 C CNN
@@
 Text Notes 8250 1300 0    60   ~ 0
 Ev version pass through\n
+$Comp
+L +3.3V #PWR011
+U 1 1 5B59ECC3
+P 8300 4600
+F 0 "#PWR011" H 8300 4450 50  0001 C CNN
+F 1 "+3.3V" H 8300 4740 50  0000 C CNN
+F 2 "" H 8300 4600 50  0001 C CNN
+F 3 "" H 8300 4600 50  0001 C CNN
+	1    8300 4600
+	1    0    0    -1
+$EndComp
+$Comp
+L +3.3V #PWR012
+U 1 1 5B59F043
+P 6100 2650
+F 0 "#PWR012" H 6100 2500 50  0001 C CNN
+F 1 "+3.3V" H 6100 2790 50  0000 C CNN
+F 2 "" H 6100 2650 50  0001 C CNN
+F 3 "" H 6100 2650 50  0001 C CNN
+	1    6100 2650
+	1    0    0    -1
+$EndComp
+Text Notes 8250 1700 0    60   ~ 0
+Annoter certaines pins (5V, 3V3, GND,...)
+Text Notes 8250 1900 0    60   ~ 0
+enlever bme280
+Text Notes 8250 2100 0    60   ~ 0
+LED RGB WS2812 WS2813
+Text Notes 8250 2300 0    60   ~ 0
+C1 en 0603  et R aussi
 Text Notes 8250 1500 0    60   ~ 0
 mesurer tension sur pin data IRM

Commit message: fix pcb v1.0 (and update to kicad v5)
Parts:
- removed DS18: DS18, Socket_Strips:Socket_Strip_Straight_1x03_Pitch2.54mm, symbol DHT11_Temperature_Humidity
- added D3: DIODE, Resistors_SMD:R_0805, symbol pspice:DIODE
- added D4: WS2813, LEDs:LED_WS2812-PLCC6, symbol LED:WS2813
- added J3, J4, J5: Pad, Wire_Pads:SolderWirePad_single_1-5mmDrill, symbol Connector:Conn_01x01_Female
- added JP1: Jumper, PTL-ino:solder-jumper-2, symbol Device:Jumper
- C1: footprint Capacitors_SMD:C_1206 -> Capacitors_SMD:C_0603_HandSoldering; symbol C -> PTL-IR_remote-rescue:C
- D1, D2: symbol IR204A -> PTL-IR_remote-rescue:IR204A
- DHT22: symbol DHT22_Temperature_Humidity -> sensors:DHT22_Temperature_Humidity
- J1, J2: symbol Conn_01x08_Male -> PTL-IR_remote-rescue:Conn_01x08_Male
- PR1: symbol R_PHOTO -> PTL-IR_remote-rescue:R_PHOTO
- Q1: symbol 2N7002 -> PTL-IR_remote-rescue:2N7002
- R1, R2, R4, R5: footprint Resistors_SMD:R_1206 -> Resistors_SMD:R_0805; symbol R -> PTL-IR_remote-rescue:R
- U1: symbol TSOP45xx -> PTL-IR_remote-rescue:TSOP45xx
- bme280: symbol Conn_01x04_Male -> PTL-IR_remote-rescue:Conn_01x04_Male
Connections:
- net labels added: D3, RX
- wire segments 51 -> 71
- no-connect marks 6 -> 8
Other:
- note added: "(5V-0.7V)*0.7 = 3.01V\nDin < 3.01V ;-)"
- note added: "Optional DS18B20\n(one wire)"
- note added: "Optional I2C\n(bme280)"
- note removed: "Annoter certaines pins (5V, 3V3, GND,...)"
- note removed: "C1 en 0603 et R aussi"
- note removed: "Corriger plan de masse"
- note removed: "Ev version pass through\n"
- note removed: "LED RGB WS2812 WS2813"
- note removed: "Optional sensors\nbme280 I2C SPI"
- note removed: "Passer sensors en 3V3"
- note removed: "enlever bme280"
- note removed: "mesurer tension sur pin data IRM"
- moved on the sheet: D1, D2, Q1, U1

Commit message: split schema
Parts:
- U1: value TSOP45xx -> TSOP4838
Connections:
- net labels added: DHT, IR, IRM, OneW, PhR, RGB
- wire segments 71 -> 66
Other:
- note added: "IR receiver"
- note added: "IR transmitter"
- note added: "RGB"
- note added: "Thermometer"
- note added: "Wemos\nheaders"
- note added: "brightness"
- note removed: "Option bme280\ndaughter shield"
- moved on the sheet: D1, D2, Q1, U1

Commit message: change diode footprint and reroute
Parts:
- C1: footprint Capacitors_SMD:C_0603_HandSoldering -> Capacitor_SMD:C_0603_1608Metric_Pad1.05x0.95mm_HandSolder
- D1, D2: footprint LEDs:LED_D3.0mm -> LED_THT:LED_D5.0mm_IRGrey
- D3: footprint Resistors_SMD:R_0805 -> Diode_SMD:D_PowerDI-123
- D4: footprint LEDs:LED_WS2812-PLCC6 -> LED_SMD:LED_WS2812_PLCC6_5.0x5.0mm_P1.6mm
- DHT22: footprint Socket_Strips:Socket_Strip_Straight_1x04_Pitch2.54mm -> Connector_PinHeader_2.54mm:PinHeader_1x04_P2.54mm_Vertical
- J1, J2: footprint Socket_Strips:Socket_Strip_Straight_1x08_Pitch2.54mm -> Connector_PinHeader_2.54mm:PinHeader_1x08_P2.54mm_Vertical
- J3, J4, J5: footprint Wire_Pads:SolderWirePad_single_1-5mmDrill -> Connector_Wire:SolderWirePad_1x01_Drill1.5mm
- PR1: footprint Socket_Strips:Socket_Strip_Straight_1x02_Pitch2.54mm -> OptoDevice:R_LDR_4.9x4.2mm_P2.54mm_Vertical
- Q1: footprint TO_SOT_Packages_SMD:SOT-23 -> Package_TO_SOT_SMD:SOT-23
- R1, R2, R4, R5: footprint Resistors_SMD:R_0805 -> Resistor_SMD:R_0805_2012Metric
- U1: footprint Opto-Devices:IRReceiver_Vishay_MOLD-3pin -> OptoDevice:Vishay_MINIMOLD-3Pin
- bme280: footprint Pin_Headers:Pin_Header_Straight_1x04_Pitch2.54mm -> Connector_PinHeader_2.54mm:PinHeader_1x04_P2.54mm_Vertical
Connections:
- net labels added: GNDREF
- net labels removed: GND
- wire segments 66 -> 65

Commit message: change led pin (D2), add jumper (bme280)
Connections:
- net labels added: D2
- net labels removed: RGB, RX
- wire segments 65 -> 64
- no-connect marks 8 -> 9
Changed lines of the file:
@@
 Wire Wire Line
 	8000 2200 8000 2350
-Wire Wire Line
-	1700 4850 1900 4850
 $Comp
 L power:+5V #PWR0101
@@
 	1    0    0    -1
 $EndComp
-Wire Wire Line
-	7350 4800 6850 4800
 Text Label 7150 4900 0    60   ~ 0
-SCL
+D2
 Text Label 7150 5000 0    60   ~ 0
 SDA
@@
 Text Label 7150 5200 0    60   ~ 0
 D4
-Text Label 7150 4800 0    60   ~ 0
-RX
 $Comp
 L pspice:DIODE D3
@@
 L Device:Jumper JP1
 U 1 1 5B5D2C34
-P 2200 4850
-F 0 "JP1" H 2200 5114 50  0000 C CNN
-F 1 "Jumper" H 2200 5023 50  0000 C CNN
-F 2 "PTL-ino:solder-jumper-2" H 2200 4850 50  0001 C CNN
-F 3 "~" H 2200 4850 50  0001 C CNN
-	1    2200 4850
+P 1850 7100
+F 0 "JP1" H 1850 7364 50  0000 C CNN
+F 1 "Jumper" H 1850 7273 50  0000 C CNN
+F 2 "PTL-ino:solder-jumper-2" H 1850 7100 50  0001 C CNN
+F 3 "~" H 1850 7100 50  0001 C CNN
+	1    1850 7100
 	1    0    0    -1
 $EndComp
@@
 Optional DS18B20\n(one wire)
 Wire Wire Line
-	1600 7000 1600 7050
+	950  7000 950  7050
 Wire Wire Line
 	6850 4900 7350 4900
@@
 $EndComp
 Wire Wire Line
-	1600 7000 2550 7000
+	950  7000 2550 7000
 $Comp
 L PTL-IR_remote-rescue:Conn_01x04_Male bme280
@@
 OneW
 Wire Wire Line
-	2500 4850 2650 4850
-Wire Wire Line
 	3100 5150 1700 5150
 Connection ~ 1700 5150
@@
 	5100 5400 5100 5350
 Text GLabel 4650 2450 0    60   Input ~ 0
-RGB
-Text GLabel 7350 4800 2    60   Output ~ 0
-RGB
+D2
 Text GLabel 7350 4900 2    60   Output ~ 0
-SCL
+D2
 Text GLabel 7350 5000 2    60   Output ~ 0
 SDA
-Text GLabel 2150 7100 0    60   Input ~ 0
-SCL
+Text GLabel 1450 7100 0    60   Input ~ 0
+D2
 Text GLabel 2150 7200 0    60   Input ~ 0
 SDA
@@
 L power:GNDREF #PWR0108
 U 1 1 5B5D9D23
-P 1600 7050
-F 0 "#PWR0108" H 1600 6800 50  0001 C CNN
-F 1 "GNDREF" H 1605 6877 50  0000 C CNN
-F 2 "" H 1600 7050 50  0001 C CNN
-F 3 "" H 1600 7050 50  0001 C CNN
-	1    1600 7050
+P 950 7050
+F 0 "#PWR0108" H 950 6800 50  0001 C CNN
+F 1 "GNDREF" H 955 6877 50  0000 C CNN
+F 2 "" H 950 7050 50  0001 C CNN
+F 3 "" H 950 7050 50  0001 C CNN
+	1    950  7050
 	1    0    0    -1
 $EndComp
@@
 	1    0    0    -1
 $EndComp
+Wire Wire Line
+	1700 4850 2650 4850
+Wire Wire Line
+	1550 7100 1450 7100
+NoConn ~ 6850 4800
+Text Label 2300 7100 0    60   ~ 0
+SCL
 $EndSCHEMATC

Commit message: replace OneWIre pads by 2.54 header
Parts:
- removed J3, J4, J5: Pad, Connector_Wire:SolderWirePad_1x01_Drill1.5mm, symbol Connector:Conn_01x01_Female
- added J4: Conn_01x03_Female, Connector_PinHeader_2.54mm:PinHeader_1x03_P2.54mm_Vertical, symbol Connector:Conn_01x03_Female
Connections:
- wire segments 64 -> 67
Changed lines of the file:
@@
 F 1 "DHT22" H 2000 3900 60  0000 C CNN
 F 2 "Connector_PinHeader_2.54mm:PinHeader_1x04_P2.54mm_Vertical" H 2000 2950 60  0001 C CNN
-F 3 " https://www.sparkfun.com/datasheets/Sensors/Temperature/DHT22.pdf" H 2000 2950 60  0000 C CNN
+F 3 " https://www.sparkfun.com/datasheets/Sensors/Temperature/DHT22.pdf" V 2000 2950 60  0001 C CNN
 	1    2000 2950
 	0    1    1    0
@@
 	10200 2100 10200 1900
 Wire Wire Line
-	1400 4850 1700 4850
-Wire Wire Line
-	1400 5450 3100 5450
+	1150 4850 1700 4850
+Wire Wire Line
+	1300 5450 3100 5450
 Text Label 5750 5100 0    60   ~ 0
 D6
@@
 	5450 2000 5450 2150
 $Comp
-L Connector:Conn_01x01_Female J4
-U 1 1 5B5C66AB
-P 1200 5450
-F 0 "J4" H 1094 5225 50  0000 C CNN
-F 1 "Pad" H 1094 5316 50  0000 C CNN
-F 2 "Connector_Wire:SolderWirePad_1x01_Drill1.5mm" H 1200 5450 50  0001 C CNN
-F 3 "~" H 1200 5450 50  0001 C CNN
-	1    1200 5450
-	-1   0    0    1
-$EndComp
-$Comp
-L Connector:Conn_01x01_Female J5
-U 1 1 5B5C7D58
-P 1200 4850
-F 0 "J5" H 1094 4625 50  0000 C CNN
-F 1 "Pad" H 1094 4716 50  0000 C CNN
-F 2 "Connector_Wire:SolderWirePad_1x01_Drill1.5mm" H 1200 4850 50  0001 C CNN
-F 3 "~" H 1200 4850 50  0001 C CNN
-	1    1200 4850
-	-1   0    0    1
-$EndComp
-$Comp
-L Connector:Conn_01x01_Female J3
-U 1 1 5B5C7EFD
-P 1200 5150
-F 0 "J3" H 1094 4925 50  0000 C CNN
-F 1 "Pad" H 1094 5016 50  0000 C CNN
-F 2 "Connector_Wire:SolderWirePad_1x01_Drill1.5mm" H 1200 5150 50  0001 C CNN
-F 3 "~" H 1200 5150 50  0001 C CNN
-	1    1200 5150
-	-1   0    0    1
-$EndComp
-$Comp
 L Device:Jumper JP1
 U 1 1 5B5D2C34
@@
 Wire Wire Line
 	1450 5150 1700 5150
-Wire Wire Line
-	1400 5150 1700 5150
 $Comp
 L power:GNDREF #PWR0106
@@
 Text Label 2300 7100 0    60   ~ 0
 SCL
+$Comp
+L Connector:Conn_01x03_Female J4
+U 1 1 5B62EF32
+P 950 4950
+F 0 "J4" H 844 4625 50  0000 C CNN
+F 1 "Conn_01x03_Female" H 844 4716 50  0000 C CNN
+F 2 "Connector_PinHeader_2.54mm:PinHeader_1x03_P2.54mm_Vertical" H 950 4950 50  0001 C CNN
+F 3 "~" H 950 4950 50  0001 C CNN
+	1    950  4950
+	-1   0    0    1
+$EndComp
+Wire Wire Line
+	1450 5150 1450 4950
+Wire Wire Line
+	1450 4950 1150 4950
+Wire Wire Line
+	1300 5450 1300 5050
+Wire Wire Line
+	1300 5050 1150 5050
 $EndSCHEMATC
