File: PTL-IR_remote.sch (KiCad schematic (older format))
At the start: 18 parts, among them J1 8p, J2 8p, J4 Conn_01x03_Female, Q1 2N7002, U1 TSOP4838

Commit message: Moved to Kicad5 Fixed swap of 5V and GND PCB is now V1.2
Parts:
- C1: symbol PTL-IR_remote-rescue:C -> Device:C
- D1, D2: symbol PTL-IR_remote-rescue:IR204A -> LED:IR204A
- DHT22: symbol sensors:DHT22_Temperature_Humidity -> Sensor:DHT11
- J1, J2: symbol PTL-IR_remote-rescue:Conn_01x08_Male -> Connector:Conn_01x08_Male
- PR1: symbol PTL-IR_remote-rescue:R_PHOTO -> Sensor_Optical:A1050
- Q1: symbol PTL-IR_remote-rescue:2N7002 -> Transistor_FET:2N7002
- R1, R2, R4, R5: symbol PTL-IR_remote-rescue:R -> Device:R
- U1: symbol PTL-IR_remote-rescue:TSOP45xx -> Interface_Optical:TSOP45xx
- bme280: symbol PTL-IR_remote-rescue:Conn_01x04_Male -> Connector:Conn_01x04_Male
Connections:
- net labels added: RGB
- net labels removed: D2
- wire segments 67 -> 70
Other:
- note added: "SCL\n"
Changed lines of the file:
@@
 $EndComp
 $Comp
-L PTL-IR_remote-rescue:IR204A D1
+L LED:IR204A D1
 U 1 1 5B433B66
 P 10200 2200
@@
 $EndComp
 $Comp
-L PTL-IR_remote-rescue:R R2
+L Device:R R2
 U 1 1 5B433CA2
 P 10200 2700
@@
 	10200 3500 10200 3400
 $Comp
-L PTL-IR_remote-rescue:C C1
+L Device:C C1
 U 1 1 5B4343A1
 P 2850 1450
@@
 	2200 1250 2850 1250
 $Comp
-L PTL-IR_remote-rescue:2N7002 Q1
+L Transistor_FET:2N7002 Q1
 U 1 1 5B48C0DB
 P 10100 3200
@@
 $EndComp
 $Comp
-L PTL-IR_remote-rescue:TSOP45xx U1
+L Interface_Optical:TSOP45xx U1
 U 1 1 5B48CD02
 P 1800 1450
@@
 Connection ~ 2850 1250
 $Comp
-L PTL-IR_remote-rescue:R_PHOTO PR1
+L Sensor_Optical:A1050 PR1
 U 1 1 5B48DA29
 P 8000 1950
@@
 $EndComp
 $Comp
-L PTL-IR_remote-rescue:R R1
+L Device:R R1
 U 1 1 5B48DE24
 P 8000 2500
@@
 	8300 2200 8000 2200
 Connection ~ 8000 2200
-Wire Wire Line
-	6850 5300 7050 5300
-Wire Wire Line
-	1600 3100 2000 3100
-$Comp
-L sensors:DHT22_Temperature_Humidity DHT22
+$Comp
+L Sensor:DHT11 DHT22
 U 1 1 5B48F14D
-P 2000 2950
-F 0 "DHT22" H 2000 4000 60  0000 C CNN
-F 1 "DHT22" H 2000 3900 60  0000 C CNN
-F 2 "Connector_PinHeader_2.54mm:PinHeader_1x04_P2.54mm_Vertical" H 2000 2950 60  0001 C CNN
-F 3 " https://www.sparkfun.com/datasheets/Sensors/Temperature/DHT22.pdf" V 2000 2950 60  0001 C CNN
-	1    2000 2950
+P 2500 2950
+F 0 "DHT22" H 2600 3350 60  0000 C CNN
+F 1 "DHT22" H 2600 3250 60  0000 C CNN
+F 2 "Connector_PinHeader_2.54mm:PinHeader_1x04_P2.54mm_Vertical" H 2500 2950 60  0001 C CNN
+F 3 " https://www.sparkfun.com/datasheets/Sensors/Temperature/DHT22.pdf" V 2500 2950 60  0001 C CNN
+	1    2500 2950
 	0    1    1    0
 $EndComp
-Wire Wire Line
-	1600 3100 1600 3250
-Wire Wire Line
-	1750 2750 1750 2800
 Text Label 5750 4800 0    60   ~ 0
 ADC
@@
 	1    0    0    -1
 $EndComp
-Wire Wire Line
-	1750 2800 2000 2800
 $Comp
 L power:+5V #PWR09
@@
 	3100 4950 3100 5150
 $Comp
-L PTL-IR_remote-rescue:R R4
+L Device:R R4
 U 1 1 5B4911B0
 P 3300 1250
@@
 	3450 1250 3550 1250
 $Comp
-L PTL-IR_remote-rescue:IR204A D2
+L LED:IR204A D2
 U 1 1 5B4AEBDC
 P 10200 1700
@@
 	10200 2100 10200 1900
 Wire Wire Line
-	1150 4850 1700 4850
-Wire Wire Line
 	1300 5450 3100 5450
 Text Label 5750 5100 0    60   ~ 0
 D6
 $Comp
-L PTL-IR_remote-rescue:R R5
+L Device:R R5
 U 1 1 5B4AFAC2
 P 1700 5000
@@
 	1    0    0    -1
 $EndComp
-Connection ~ 1700 4850
 $Bitmap
 Pos 10500 6850
@@
 $EndBitmap
 $Comp
-L PTL-IR_remote-rescue:Conn_01x08_Male J1
+L Connector:Conn_01x08_Male J1
 U 1 1 5B4B47C9
 P 6200 5100
@@
 $EndComp
 $Comp
-L PTL-IR_remote-rescue:Conn_01x08_Male J2
+L Connector:Conn_01x08_Male J2
 U 1 1 5B4B4972
 P 6650 5000
@@
 L power:+3.3V #PWR011
 U 1 1 5B59ECC3
-P 1750 2750
-F 0 "#PWR011" H 1750 2600 50  0001 C CNN
-F 1 "+3.3V" H 1750 2890 50  0000 C CNN
-F 2 "" H 1750 2750 50  0001 C CNN
-F 3 "" H 1750 2750 50  0001 C CNN
-	1    1750 2750
+P 3050 2750
+F 0 "#PWR011" H 3050 2600 50  0001 C CNN
+F 1 "+3.3V" H 3050 2890 50  0000 C CNN
+F 2 "" H 3050 2750 50  0001 C CNN
+F 3 "" H 3050 2750 50  0001 C CNN
+	1    3050 2750
 	1    0    0    -1
 $EndComp
@@
 $EndComp
 Text Label 7150 4900 0    60   ~ 0
-D2
+SCL
 Text Label 7150 5000 0    60   ~ 0
 SDA
@@
 	950  7000 2550 7000
 $Comp
-L PTL-IR_remote-rescue:Conn_01x04_Male bme280
+L Connector:Conn_01x04_Male bme280
 U 1 1 5B48E4DC
 P 2750 7100
@@
 $EndComp
 Wire Wire Line
-	7800 5500 7800 5400
+	7800 5500 7800 5450
 $Comp
 L LED:WS2813 D4
@@
 Text GLabel 5700 5100 0    60   BiDi ~ 0
 OneW
-Wire Wire Line
-	3100 5150 1700 5150
-Connection ~ 1700 5150
 $Comp
 L power:+3.3V #PWR0104
@@
 	5100 5400 5100 5350
 Text GLabel 4650 2450 0    60   Input ~ 0
-D2
-Text GLabel 7350 4900 2    60   Output ~ 0
-D2
+RGB
+Text GLabel 7350 5200 2    60   Output ~ 0
+RGB
 Text GLabel 7350 5000 2    60   Output ~ 0
 SDA
-Text GLabel 1450 7100 0    60   Input ~ 0
-D2
 Text GLabel 2150 7200 0    60   Input ~ 0
 SDA
@@
 Wire Wire Line
 	1950 6900 2350 6900
-Text GLabel 7350 5200 2    60   Input ~ 0
+Text GLabel 7350 4900 2    60   Input ~ 0
 DHT
-Text GLabel 1750 2900 0    60   Output ~ 0
+Text GLabel 2500 3400 3    60   Output ~ 0
 DHT
 Wire Wire Line
-	1750 2900 2000 2900
-Wire Wire Line
 	7350 5200 6850 5200
-Wire Wire Line
-	6850 5400 7800 5400
-Wire Wire Line
-	7050 5300 7050 5800
 Wire Wire Line
 	7050 5800 7350 5800
@@
 Text Notes 9950 1000 0    60   ~ 0
 IR transmitter
-Wire Wire Line
-	1450 5150 1700 5150
 $Comp
 L power:GNDREF #PWR0106
@@
 L power:GNDREF #PWR0109
 U 1 1 5B5D9DBE
-P 1600 3250
-F 0 "#PWR0109" H 1600 3000 50  0001 C CNN
-F 1 "GNDREF" H 1605 3077 50  0000 C CNN
-F 2 "" H 1600 3250 50  0001 C CNN
-F 3 "" H 1600 3250 50  0001 C CNN
-	1    1600 3250
+P 2100 2950
+F 0 "#PWR0109" H 2100 2700 50  0001 C CNN
+F 1 "GNDREF" H 2105 2777 50  0000 C CNN
+F 2 "" H 2100 2950 50  0001 C CNN
+F 3 "" H 2100 2950 50  0001 C CNN
+	1    2100 2950
 	1    0    0    -1
 $EndComp
@@
 	1    0    0    -1
 $EndComp
-Connection ~ 7800 5400
 $Comp
 L power:GNDREF #PWR0103
@@
 	1    0    0    -1
 $EndComp
-Wire Wire Line
-	1700 4850 2650 4850
-Wire Wire Line
-	1550 7100 1450 7100
 NoConn ~ 6850 4800
-Text Label 2300 7100 0    60   ~ 0
-SCL
 $Comp
 L Connector:Conn_01x03_Female J4
@@
 Wire Wire Line
 	1300 5050 1150 5050
+Wire Wire Line
+	1150 4850 1700 4850
+Wire Wire Line
+	1450 5150 1700 5150
+Wire Wire Line
+	2500 3250 2500 3400
+Wire Wire Line
+	2200 2850 2100 2850
+Wire Wire Line
+	2100 2850 2100 2950
+Wire Wire Line
+	2800 2850 3050 2850
+Wire Wire Line
+	3050 2850 3050 2750
+Connection ~ 1700 4850
+Wire Wire Line
+	1700 4850 2650 4850
+Connection ~ 1700 5150
+Wire Wire Line
+	1700 5150 3100 5150
+Wire Wire Line
+	1550 7100 1250 7100
+Text GLabel 1250 7100 0    60   Output ~ 0
+DHT
+Text Notes 2400 7100 0    60   ~ 0
+SCL\n
+Wire Wire Line
+	7050 5800 7050 5400
+Wire Wire Line
+	7050 5400 6850 5400
+Wire Wire Line
+	6850 5300 7700 5300
+Wire Wire Line
+	7700 5300 7700 5450
+Wire Wire Line
+	7700 5450 7800 5450
+Connection ~ 7800 5450
+Wire Wire Line
+	7800 5450 7800 5400
 $EndSCHEMATC
